File: 1.PCB/node.brd (EAGLE design)
At the start: 48.3 x 96.2 mm, 16 parts, among them IC1 7805TV

Commit message: changes done
Connections:
- net D3 renamed RX_GPS
- net D4 renamed TX_GPS
Changed lines of the file:
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@@
 <drawing>
 <settings>
-<setting alwaysvectorfont="yes"/>
+<setting alwaysvectorfont="no"/>
 <setting verticaltext="up"/>
 </settings>
@@
 <wire x1="36.068" y1="38.735" x2="39.497" y2="38.735" width="0.762" layer="16"/>
 </signal>
-<signal name="D4">
+<signal name="TX_GPS">
 <contactref element="ARDUINO_NANO1" pad="22"/>
 <contactref element="SV2" pad="9"/>
@@
 <wire x1="20.701" y1="56.642" x2="20.828" y2="56.515" width="0.762" layer="16"/>
 </signal>
-<signal name="D3">
+<signal name="RX_GPS">
 <contactref element="ARDUINO_NANO1" pad="21"/>
 <contactref element="SV2" pad="10"/>
