File: 1.PCB/node.sch (EAGLE design)
At the start: 16 parts, among them IC1 7805TV

Commit message: changes done
Connections:
- net D3 renamed RX_GPS
- net D4 renamed TX_GPS
Changed lines of the file:
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@@
 <drawing>
 <settings>
-<setting alwaysvectorfont="yes"/>
+<setting alwaysvectorfont="no"/>
 <setting verticaltext="up"/>
 </settings>
@@
 </segment>
 </net>
-<net name="D4" class="0">
+<net name="TX_GPS" class="0">
 <segment>
 <pinref part="ARDUINO_NANO1" gate="G$1" pin="D4"/>
@@
 </segment>
 </net>
-<net name="D3" class="0">
+<net name="RX_GPS" class="0">
 <segment>
 <pinref part="ARDUINO_NANO1" gate="G$1" pin="D3"/>
